Commit message: 20220227_8点対応

File: damitora_description/urdf/damitora_copy.urdf (robot description, URDF)
Before this commit: robot seto_scararobot, 18 links, 17 joints
Links:
- removed link tracker_L_link2
- removed link tracker_R_link2
Joints:
- removed joint fixed_tracker_L2
- removed joint fixed_tracker_R2
- joint L_lower_leg_P: limit lower=-3.14159 upper=0 effort=1000.0 velocity=2.0 -> lower=-3.14159 upper=3.14159 effort=1000.0 velocity=2.0
- joint R_lower_leg_P: limit lower=0 upper=3.14159 effort=1000.0 velocity=2.0 -> lower=-3.14159 upper=3.14159 effort=1000.0 velocity=2.0
