Commit message: 20220624

File: damitora_description/urdf/damitora_5_1.urdf (robot description, URDF)
Before this commit: robot seto_scararobot, 20 links, 19 joints
Links:
- removed link Foot_L_link
- removed link Foot_R_link
- link lower_leg_L_link: geometry visual mesh filename=package://damitora_description/meshes/lower_leg.stl
- link lower_leg_R_link: geometry visual mesh filename=package://damitora_description/meshes/lower_leg.stl
Joints:
- removed joint L_foot_P
- removed joint R_foot_P
- joint fixed_tracker_L: origin xyz=0.012 0 0.002 rpy=0 -1.3 0 -> xyz=0.005 0 -0.04 rpy=0 0 0; parent Foot_L_link -> lower_leg_L_link
- joint fixed_tracker_R: origin xyz=0.012 0 0.002 rpy=0 -1.3 0 -> xyz=0.005 0 -0.04 rpy=0 0 0; parent Foot_R_link -> lower_leg_R_link
